File: raspberry-tart-hat/hat.kicad_sch (KiCad schematic)
At the start: 10 parts, among them J1 40HAT, J2 HDR_WP, U1 CAT24C32

Commit message: Initial pcb layout complete
Parts:
- R1, R2, R3, U1: Supplier JLCPCB -> LCSC
Connections:
- net P3V3 is gone; now on net 3V3: R1.2, R2.1, R3.1, U1.8 (VCC)
Changed lines of the file:
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@@
     (effects (font (size 1.27 1.27)) (justify right bottom))
-  )
-  (label "P3V3" (at 120.65 72.39 180)
-    (effects (font (size 1.524 1.524)) (justify right bottom))
   )
   (label "PCM_CLK" (at 224.79 76.2 180)
@@
   (label "GPIO_27" (at 158.75 78.74 0)
     (effects (font (size 1.27 1.27)) (justify left bottom))
+  )
+  (label "P3V3_HAT" (at 120.65 72.39 180)
+    (effects (font (size 1.524 1.524)) (justify right bottom))
   )
   (label "TXD" (at 102.87 149.86 180)
@@
       (effects (font (size 1.27 1.27)) hide)
     )
-    (property "Supplier" "JLCPCB" (id 7) (at 105.41 74.93 0)
+    (property "Supplier" "LCSC" (id 7) (at 105.41 74.93 0)
       (effects (font (size 1.27 1.27)) hide)
     )
@@
       (effects (font (size 1.27 1.27)) hide)
     )
-    (property "Supplier" "JLCPCB" (id 7) (at 128.27 86.36 0)
+    (property "Supplier" "LCSC" (id 7) (at 128.27 86.36 0)
       (effects (font (size 1.27 1.27)) hide)
     )
@@
     (property "Reference" "J1" (id 0) (at 200.66 60.96 0))
     (property "Value" "40HAT" (id 1) (at 184.15 60.96 0))
-    (property "Footprint" "Connector_PinSocket_2.54mm:PinSocket_2x20_P2.54mm_Vertical" (id 2) (at 191.77 58.42 0))
-    (property "Datasheet" "https://media.digikey.com/pdf/Data%20Sheets/Sullins%20PDFs/Female_Headers.100_DS.pdf" (id 3) (at 173.99 63.5 0))
+    (property "Footprint" "Connector_PinSocket_2.54mm:PinSocket_2x20_P2.54mm_Vertical" (id 2) (at 191.77 58.42 0)
+      (effects (font (size 1.27 1.27)) hide)
+    )
+    (property "Datasheet" "https://media.digikey.com/pdf/Data%20Sheets/Sullins%20PDFs/Female_Headers.100_DS.pdf" (id 3) (at 173.99 63.5 0)
+      (effects (font (size 1.27 1.27)) hide)
+    )
     (property "Manufacturer" "Sullins Connector Solutions" (id 4) (at 191.77 63.5 0)
       (effects (font (size 1.27 1.27)) hide)
@@
       (effects (font (size 1.27 1.27)) hide)
     )
-    (property "Supplier" "JLCPCB" (id 7) (at 134.62 86.36 0)
+    (property "Supplier" "LCSC" (id 7) (at 134.62 86.36 0)
       (effects (font (size 1.27 1.27)) hide)
     )
@@
       (effects (font (size 1.27 1.27)) hide)
     )
-    (property "Supplier" "JLCPCB" (id 6) (at 113.03 90.17 0)
-      (effects (font (size 1.27 1.27)) hide)
-    )
+    (property "Supplier" "LCSC" (id 6) (at 113.03 90.17 0)
+      (effects (font (size 1.27 1.27)) hide)
+    )
