File: raspberry-tart-hat/raspberry-tart-hat.kicad_pcb (KiCad board)
At the start: 2 copper layers, 0 parts

Commit message: Initial pcb layout complete
Parts:
- added C1: 10n, Capacitor_SMD:C_0805_2012Metric, F.Cu at (152.7, 84.2)
- added C2: 10n, Capacitor_SMD:C_0805_2012Metric, F.Cu at (156.1, 84.2)
- added C3: 100n, Capacitor_SMD:C_0805_2012Metric, F.Cu at (148.8, 86.9)
- added D1: LED_PWR, LED_SMD:LED_0603_1608Metric, F.Cu at (136.8, 88.0)
- added D2: LED_RX, LED_SMD:LED_0603_1608Metric, F.Cu at (136.8, 89.7)
- added D3: LED_TX, LED_SMD:LED_0603_1608Metric, F.Cu at (136.8, 91.3)
- added D4: 1N4148WS, Diode_SMD:D_SOD-323, F.Cu at (148.8, 90.5)
- added D5: 1N4148WS, Diode_SMD:D_SOD-323, F.Cu at (160.0, 90.6)
- added G***: LOGO, LOGO, F.Cu at (183.9, 90.6)
- added H1: 3mm, MountingHole:MountingHole_3mm, F.Cu at (130.0, 80.0)
- added H2: 3mm, MountingHole:MountingHole_3mm, F.Cu at (188.0, 80.0)
- added H3: 3mm, MountingHole:MountingHole_3mm, F.Cu at (188.0, 129.0)
- added H4: 3mm, MountingHole:MountingHole_3mm, F.Cu at (130.0, 129.0)
- added J1: 40HAT, Connector_PinSocket_2.54mm:PinSocket_2x20_P2.54mm_Vertical, B.Cu at (134.9, 81.3)
- added J2: HDR_WP, Connector_PinHeader_2.54mm:PinHeader_1x03_P2.54mm_Vertical, F.Cu at (167.2, 92.0)
- added J3: JST_SH_SWD, Connector_JST:JST_SH_BM03B-SRSS-TB_1x03-1MP_P1.00mm_Vertical, F.Cu at (185.1, 105.8)
- added J7: HDR_PICO, Connector_PinSocket_2.54mm:PinSocket_2x20_P2.54mm_Vertical, F.Cu at (134.9, 124.9)
- added Q1: DMG2305UX, Package_TO_SOT_SMD:SOT-23, F.Cu at (128.6, 92.3)
- added R1: 1k, Resistor_SMD:R_1206_3216Metric, F.Cu at (164.6, 88.5)
- added R2: 3k9, Resistor_SMD:R_0805_2012Metric, F.Cu at (165.2, 86.4)
- added R3: 3k9, Resistor_SMD:R_0805_2012Metric, F.Cu at (165.2, 84.3)
- added R4: 330, Resistor_SMD:R_0603_1608Metric, F.Cu at (133.7, 89.7)
- added R5: 1M, Resistor_SMD:R_0603_1608Metric, F.Cu at (152.7, 86.0)
- added R7: 330, Resistor_SMD:R_0603_1608Metric, F.Cu at (133.7, 91.3)
- added R8: 1M, Resistor_SMD:R_0603_1608Metric, F.Cu at (156.0, 86.0)
- added R9: 330, Resistor_SMD:R_0603_1608Metric, F.Cu at (140.0, 88.0)
- added U1: CAT24C32, Package_SO:SOIC-8_3.9x4.9mm_P1.27mm, F.Cu at (170.7, 87.1)
- added U2: Pico, MCU_RaspberryPi_and_Boards:RPi_Pico_SMD_TH, F.Cu at (151.5, 105.7)
- added U3: 74HC14, Package_SO:SOIC-14_3.9x8.7mm_P1.27mm, F.Cu at (154.4, 90.5)
Routing:
- net GND: track 0.00 -> 180.5 mm, vias 0 -> 11
- net /TXD_PI: track 0.00 -> 72.8 mm, vias 0 -> 2
- net /RXD_PI: track 0.00 -> 65.9 mm, vias 0 -> 1
- net /UART_GND: track 0.00 -> 59.2 mm
- net /SWDIO: track 0.00 -> 54.6 mm
- net /SWD_GND: track 0.00 -> 51.1 mm
- net /SWCLK: track 0.00 -> 48.6 mm
- net +3V3: track 0.00 -> 47.8 mm, vias 0 -> 1
- net /VSYS: track 0.00 -> 35.0 mm
- net /VBUS: track 0.00 -> 34.9 mm
- net /GPIO16: track 0.00 -> 32.9 mm
- net /GPIO26: track 0.00 -> 31.3 mm
- net /GPIO18: track 0.00 -> 31.3 mm
- net /RUN: track 0.00 -> 31.3 mm
- net /GPIO27: track 0.00 -> 31.3 mm
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- added copper zone on F.Cu, net +5V
- added copper zone on B.Cu, net GND
- added copper zone on F.Cu, net GND
Other:
- board outline added: 66 x 57 mm
- board text added: "Design: Greg Coonrod"
- board text added: "PWR"
- board text added: "RX"
- board text added: "SWD"
- board text added: "TART"
- board text added: "TX"
- board text added: "W"
- board text added: "WP"
- board text added: "rev 0"
