File: raspberry-tart-hat/raspberry-tart-hat.kicad_sch (KiCad schematic)
At the start: 0 parts

Commit message: Initial schematic complete.
Parts:
- added C1, C2: 10n, Capacitor_SMD:C_0805_2012Metric, symbol Device:C
- added C3: 100n, Capacitor_SMD:C_0805_2012Metric, symbol Device:C
- added D1: LED_PWR, LED_SMD:LED_0603_1608Metric, symbol Device:LED
- added D2: LED_RX, LED_SMD:LED_0603_1608Metric, symbol Device:LED
- added D3: LED_TX, LED_SMD:LED_0603_1608Metric, symbol Device:LED
- added D4, D5: 1N4148WS, Diode_SMD:D_SOD-323, symbol Diode:1N4448WS
- added J3: JST_SH_SWD, Connector_JST:JST_SH_BM03B-SRSS-TB_1x03-1MP_P1.00mm_Vertical, symbol Connector_Generic:Conn_01x03
- added J4, J5: HDR_20, Connector_PinSocket_2.54mm:PinSocket_1x20_P2.54mm_Vertical, symbol Connector_Generic:Conn_01x20
- added J6: HDR_3, Connector_PinSocket_2.54mm:PinSocket_1x03_P2.54mm_Vertical, symbol Connector_Generic:Conn_01x03
- added JP1: DNP, symbol Jumper:Jumper_2_Open
- added Q1: DMG2305UX, Package_TO_SOT_SMD:SOT-23, symbol raspberrrypi_hat-cache:DMG2305UX
- added R4, R7, R9: 330, Resistor_SMD:R_0603_1608Metric, symbol Device:R
- added R5, R8: 1M, Resistor_SMD:R_0603_1608Metric, symbol Device:R
- added U2: Pico, MCU_RaspberryPi_and_Boards:RPi_Pico_SMD_TH, symbol MCU_RaspberryPi_and_Boards:Pico
- added U3: 74HC14, Package_SO:SOIC-14_3.9x8.7mm_P1.27mm, symbol 74xx:74HC14
Connections:
- new net: D5.2 (A), U3.6
- new net: C1.1, D4.1 (K), R5.2, U3.3
- new net: D4.2 (A), U3.2
- new net: D2.1 (K), U3.4
- new net: D1.1 (K), R9.2
- new net: C2.1, D5.1 (K), R8.2, U3.9
- new net: D2.2 (A), R4.1
- new net: D3.1 (K), U3.8
- new net: D3.2 (A), R7.1
- new net +5V: C3.1, D1.2 (A), Q1.3 (D), R4.2, R7.2, U3.14 (VCC)
- new net GND: C1.2, C2.2, C3.2, R5.1, R8.1, R9.1, U2.13 (GND), U2.18 (GND), U2.23 (GND), U2.28 (GND), U2.33 (AGND), U2.38 (GND), U2.8 (GND), U3.11, U3.13, U3.7 (GND)
- new net RXD_PI: U2.1 (GPIO0), U3.1
- new net SWCLK: J3.1 (Pin_1), U2.41 (SWCLK)
- new net SWDIO: J3.3 (Pin_3), U2.43 (SWDIO)
- new net SWD_GND: J3.2 (Pin_2), U2.42 (GND)
- new net TXD_PI: U2.2 (GPIO1), U3.5
- new net UART_GND: U2.3 (GND)
- new net VBUS: Q1.1 (G), U2.40 (VBUS)
- new net VSYS: Q1.2 (S), U2.39 (VSYS)
- no-connect marks 0 -> 75
Other:
- added sheet HAT (hat.kicad_sch)

Commit message: Initial pcb layout complete
Parts:
- added J7: HDR_PICO, Connector_PinSocket_2.54mm:PinSocket_2x20_P2.54mm_Vertical, symbol Connector_Generic:Conn_02x20_Odd_Even
- C1, C2, C3, D1, D2, D3, D4, D5, J3, Q1, R4, R5, R7, R8, R9, U3: Supplier JLCPCB -> LCSC
Connections:
- net GND: now also U3.3, J7.16 (Pin_16), J7.25 (Pin_25), J7.26 (Pin_26), J7.35 (Pin_35), J7.36 (Pin_36), J7.5 (Pin_5); no longer U2.33 (AGND), U3.13
- net RXD_PI: now also J7.2 (Pin_2)
- net TXD_PI: now also J7.4 (Pin_4)
- net UART_GND: now also J7.6 (Pin_6)
- net VBUS: now also J7.1 (Pin_1)
- net VSYS: now also J7.3 (Pin_3)
- net at C1.1, D4.1 (K), R5.2: now also U3.13; no longer U3.3
- net at D2.1 (K): now also U3.12; no longer U3.4
- net GPIO7: now reaches U2.10 (GPIO7)
- net GPIO7: now also J7.20 (Pin_20)
- net GPIO8: now reaches U2.11 (GPIO8)
- net GPIO8: now also J7.22 (Pin_22)
- net GPIO9: now reaches U2.12 (GPIO9)
- net GPIO9: now also J7.24 (Pin_24)
- net GPIO10: now reaches U2.14 (GPIO10)
- net GPIO10: now also J7.28 (Pin_28)
- net GPIO11: now reaches U2.15 (GPIO11)
- net GPIO11: now also J7.30 (Pin_30)
- net GPIO12: now reaches U2.16 (GPIO12)
- net GPIO12: now also J7.32 (Pin_32)
- net GPIO13: now reaches U2.17 (GPIO13)
- net GPIO13: now also J7.34 (Pin_34)
- net GPIO14: now reaches U2.19 (GPIO14)
- net GPIO14: now also J7.38 (Pin_38)
- net GPIO15: now reaches U2.20 (GPIO15)
- net GPIO15: now also J7.40 (Pin_40)
- net GPIO16: now reaches U2.21 (GPIO16)
- net GPIO16: now also J7.39 (Pin_39)
- net GPIO17: now reaches U2.22 (GPIO17)
- net GPIO17: now also J7.37 (Pin_37)
- net GPIO18: now reaches U2.24 (GPIO18)
- net GPIO18: now also J7.33 (Pin_33)
- net GPIO19: now reaches U2.25 (GPIO19)
- net GPIO19: now also J7.31 (Pin_31)
- net GPIO20: now reaches U2.26 (GPIO20)
- net GPIO20: now also J7.29 (Pin_29)
- net GPIO21: now reaches U2.27 (GPIO21)
- net GPIO21: now also J7.27 (Pin_27)
- net GPIO22: now reaches U2.29 (GPIO22)
- net GPIO22: now also J7.23 (Pin_23)
- net RUN: now reaches U2.30 (RUN)
- net RUN: now also J7.21 (Pin_21)
- net GPIO26: now reaches U2.31 (GPIO26_ADC0)
- net GPIO26: now also J7.19 (Pin_19)
- net GPIO27: now reaches U2.32 (GPIO27_ADC1)
- net GPIO27: now also J7.17 (Pin_17)
- net GPIO28: now reaches U2.34 (GPIO28_ADC2)
- net GPIO28: now also J7.13 (Pin_13)
- net ADC_VREF: now reaches U2.35 (ADC_VREF)
- net ADC_VREF: now also J7.11 (Pin_11)
- net 3V3: now reaches U2.36 (3V3)
- net 3V3: now also J7.9 (Pin_9)
- net 3V3_EN: now reaches U2.37 (3V3_EN)
- net 3V3_EN: now also J7.7 (Pin_7)
- net GPIO2: now reaches U2.4 (GPIO2)
- net GPIO2: now also J7.8 (Pin_8)
- net GPIO3: now reaches U2.5 (GPIO3)
- net GPIO3: now also J7.10 (Pin_10)
- net GPIO4: now reaches U2.6 (GPIO4)
- net GPIO4: now also J7.12 (Pin_12)
- net GPIO5: now reaches U2.7 (GPIO5)
- net GPIO5: now also J7.14 (Pin_14)
- net GPIO6: now reaches U2.9 (GPIO6)
- net GPIO6: now also J7.18 (Pin_18)
- new net AGND: J7.15 (Pin_15), U2.33 (AGND)
- no-connect marks 75 -> 47
